File: pumper/audio.kicad_sch (KiCad schematic)
At the start: 33 parts, among them J3 AudioJack4, U6 OPA1652AIDR, U7 PCM5102A, U8 OPA1622IDRCR

Commit message: feat: update kicad source files
Parts:
- renumbered C44 to C31, C31 to C32, C32 to C33, C33 to C34, C34 to C35, C35 to C36, C36 to C37, C37 to C38, C38 to C39, C39 to C40, C40 to C41, C41 to C42, C42 to C43, C43 to C44, D4 to D2, D5 to D3
Changed lines of the file:
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@@
 		(dnp no)
 		(fields_autoplaced yes)
-		(property "Reference" "C34"
+		(property "Reference" "C35"
 			(at 96.52 78.7399 0)
 			(effects
@@
 			(project ""
 				(path "/ff072219-444d-4fc6-9bb4-21a48733c6c1/a3b96776-b2c3-4a94-9d20-380673bf4b45"
-					(reference "C34")
+					(reference "C35")
 					(unit 1)
 				)
@@
 		(dnp no)
 		(fields_autoplaced yes)
-		(property "Reference" "C32"
+		(property "Reference" "C33"
 			(at 184.15 54.6099 0)
 			(effects
@@
 			(project "airnote"
 				(path "/ff072219-444d-4fc6-9bb4-21a48733c6c1/a3b96776-b2c3-4a94-9d20-380673bf4b45"
-					(reference "C32")
+					(reference "C33")
 					(unit 1)
 				)
@@
 		(dnp no)
 		(fields_autoplaced yes)
-		(property "Reference" "C39"
+		(property "Reference" "C40"
 			(at 88.9 96.5199 0)
 			(effects
@@
 			(project "airnote"
 				(path "/ff072219-444d-4fc6-9bb4-21a48733c6c1/a3b96776-b2c3-4a94-9d20-380673bf4b45"
-					(reference "C39")
+					(reference "C40")
 					(unit 1)
 				)
@@
 		(dnp no)
 		(fields_autoplaced yes)
-		(property "Reference" "C36"
+		(property "Reference" "C37"
 			(at 83.82 83.8199 0)
 			(effects
@@
 			(project "airnote"
 				(path "/ff072219-444d-4fc6-9bb4-21a48733c6c1/a3b96776-b2c3-4a94-9d20-380673bf4b45"
-					(reference "C36")
+					(reference "C37")
 					(unit 1)
 				)
@@
 		(dnp no)
 		(fields_autoplaced yes)
-		(property "Reference" "C31"
+		(property "Reference" "C32"
 			(at 45.72 40.6399 0)
 			(effects
@@
 			(project "airnote"
 				(path "/ff072219-444d-4fc6-9bb4-21a48733c6c1/a3b96776-b2c3-4a94-9d20-380673bf4b45"
-					(reference "C31")
+					(reference "C32")
 					(unit 1)
 				)
@@
 		(dnp no)
 		(fields_autoplaced yes)
-		(property "Reference" "C42"
+		(property "Reference" "C43"
 			(at 243.84 116.8399 0)
 			(effects
@@
 			(project ""
 				(path "/ff072219-444d-4fc6-9bb4-21a48733c6c1/a3b96776-b2c3-4a94-9d20-380673bf4b45"
-					(reference "C42")
+					(reference "C43")
 					(unit 1)
 				)
@@
 		(dnp no)
 		(fields_autoplaced yes)
-		(property "Reference" "C44"
+		(property "Reference" "C31"
 			(at 40.64 40.6399 0)
 			(effects
@@
 			(project ""
 				(path "/ff072219-444d-4fc6-9bb4-21a48733c6c1/a3b96776-b2c3-4a94-9d20-380673bf4b45"
-					(reference "C44")
+					(reference "C31")
 					(unit 1)
 				)
@@
 		(dnp no)
 		(fields_autoplaced yes)
-		(property "Reference" "D5"
+		(property "Reference" "D3"
 			(at 156.21 166.3699 90)
 			(effects
@@
 			(project ""
 				(path "/ff072219-444d-4fc6-9bb4-21a48733c6c1/a3b96776-b2c3-4a94-9d20-380673bf4b45"
-					(reference "D5")
+					(reference "D3")
 					(unit 1)
 				)
@@
 		(dnp no)
 		(fields_autoplaced yes)
-		(property "Reference" "C40"
+		(property "Reference" "C41"
 			(at 82.55 100.3299 0)
 			(effects
@@
 			(project "airnote"
 				(path "/ff072219-444d-4fc6-9bb4-21a48733c6c1/a3b96776-b2c3-4a94-9d20-380673bf4b45"
-					(reference "C40")
+					(reference "C41")
 					(unit 1)
 				)
@@
 		(dnp no)
 		(fields_autoplaced yes)
-		(property "Reference" "D4"
+		(property "Reference" "D2"
 			(at 147.32 166.3699 90)
 			(effects
@@
 			(project "airnote"
 				(path "/ff072219-444d-4fc6-9bb4-21a48733c6c1/a3b96776-b2c3-4a94-9d20-380673bf4b45"
-					(reference "D4")
+					(reference "D2")
 					(unit 1)
 				)
@@
 		(dnp no)
 		(fields_autoplaced yes)
-		(property "Reference" "C38"
+		(property "Reference" "C39"
 			(at 252.73 91.4399 0)
 			(effects
@@
 			(project "airnote"
 				(path "/ff072219-444d-4fc6-9bb4-21a48733c6c1/a3b96776-b2c3-4a94-9d20-380673bf4b45"
-					(reference "C38")
+					(reference "C39")
 					(unit 1)
 				)
@@
 		(dnp no)
 		(fields_autoplaced yes)
-		(property "Reference" "C43"
+		(property "Reference" "C44"
 			(at 252.73 116.8399 0)
 			(effects
@@
 			(project "airnote"
 				(path "/ff072219-444d-4fc6-9bb4-21a48733c6c1/a3b96776-b2c3-4a94-9d20-380673bf4b45"
-					(reference "C43")
+					(reference "C44")
 					(unit 1)
 				)
@@
 		(dnp no)
 		(fields_autoplaced yes)
-		(property "Reference" "C37"
+		(property "Reference" "C38"
 			(at 243.84 91.4399 0)
 			(effects
@@
 			(project ""
 				(path "/ff072219-444d-4fc6-9bb4-21a48733c6c1/a3b96776-b2c3-4a94-9d20-380673bf4b45"
-					(reference "C37")
+					(reference "C38")
 					(unit 1)
 				)
@@
 		(dnp no)
 		(fields_autoplaced yes)
-		(property "Reference" "C35"
+		(property "Reference" "C36"
 			(at 110.49 78.7399 0)
 			(effects
@@
 			(project "airnote"
 				(path "/ff072219-444d-4fc6-9bb4-21a48733c6c1/a3b96776-b2c3-4a94-9d20-380673bf4b45"
-					(reference "C35")
+					(reference "C36")
 					(unit 1)
 				)
@@
 		(dnp no)
 		(fields_autoplaced yes)
-		(property "Reference" "C41"
+		(property "Reference" "C42"
 			(at 184.15 111.7599 0)
 			(effects
@@
 			(project "airnote"
 				(path "/ff072219-444d-4fc6-9bb4-21a48733c6c1/a3b96776-b2c3-4a94-9d20-380673bf4b45"
-					(reference "C41")
+					(reference "C42")
 					(unit 1)
 				)
@@
 		(on_board yes)
 		(dnp no)
-		(property "Reference" "C33"
+		(property "Reference" "C34"
 			(at 193.04 54.6099 0)
 			(effects
@@
 			(project "airnote"
 				(path "/ff072219-444d-4fc6-9bb4-21a48733c6c1/a3b96776-b2c3-4a94-9d20-380673bf4b45"
-					(reference "C33")
+					(reference "C34")
 					(unit 1)
 				)

Commit message: feat: update design files
Parts:
- added R14, R15: 2kΩ, PCM_JLCPCB:R_0402, symbol PCM_JLCPCB-Resistors:0402,2kΩ
- FB1: symbol PCM_JLCPCB-Inductors:Ferrite,0603 -> PCM_JLCPCB-Inductors:Ferrite,0603,(2); Attrition Qty 6 -> 10; Current Rating 200mA -> 2A; DC Resistance 450mΩ -> 50mΩ; Impedance @ Frequency 600Ω@100MHz -> 120Ω@100MHz; LCSC C1002 -> C14709; Manufacturer Sunlord -> Murata Electronics; Part GZ1608D601TF -> BLM18PG121SN1D; Price 0.010USD -> 0.009USD; Stock 789150 -> 222675
- renumbered C27 to C30, C28 to C31, C29 to C32, C30 to C33, C31 to C34, C32 to C35, C33 to C36, C34 to C37, C35 to C38, C36 to C39, C37 to C40, C38 to C41, C39 to C42, C40 to C43, C41 to C44, C42 to C45, C43 to C46, C44 to C47, D2 to D4, D3 to D5, J3 to J2, R14 to R16, R15 to R17, R16 to R18, R17 to R19, R18 to R20, R19 to R21, R20 to R22
Connections:
- net 5102OUTL: now also R15.1
- net 5102OUTR: now also R14.1
- net GND: now also R14.2, R15.2
Other:
- note added: "OPA1652 (op-amp)"
- note removed: "OPA2141 (op-amp)"
