File: pumper/2354a.kicad_sch (KiCad schematic)
At the start: 28 parts, among them J2 Conn_01x03, SW1 1TS015A-1400-0600-CT, SW2 1TS015A-1400-0600-CT, U4 RP2354A-QFN60, U5 ABM8-272-T3_C20625731

Commit message: feat: update design files
Parts:
- removed J2: Conn_01x03, Connector_PinHeader_2.54mm:PinHeader_1x03_P2.54mm_Vertical, symbol Connector_Generic:Conn_01x03
- added C27, C28: 100nF, PCM_JLCPCB:C_0402, symbol PCM_JLCPCB-Capacitors:0402,100nF
- added D2, D3: WS2812B, PCM_JLCPCB:LED-SMD_4P-L1.6-W1.5_XL-1615RGBC-WS2812B, symbol PCM_JLCPCB-Extended:LED, WS2812B, 1615
- added TP8, TP9: TestPoint, TestPoint:TestPoint_Pad_D1.5mm, symbol Connector:TestPoint
- renumbered C11 to C12, C12 to C13, C13 to C14, C14 to C15, C15 to C16, C16 to C17, C17 to C18, C18 to C19, C19 to C20, C20 to C21, C21 to C22, C22 to C23, C23 to C24, C24 to C25, C25 to C26, C26 to C29
Connections:
- net GND: now also C27.2, C28.2, D2.3 (GND), D3.3 (GND)
- net GP12: now also D2.4 (DIN)
- net SWCLK: now also TP8.1
- net SWDIO: now also TP9.1
- new net: D2.1 (DOUT), D3.4 (DIN)
- new net VBUS: C27.1, C28.1, D2.2 (VDD), D3.2 (VDD)
Other:
- note added: "RGB LED indicator"

Commit message: feat: update kicad files
Parts:
- removed C27, C28: 100nF, PCM_JLCPCB:C_0402, symbol PCM_JLCPCB-Capacitors:0402,100nF
- removed D2, D3: WS2812B, PCM_JLCPCB:LED-SMD_4P-L1.6-W1.5_XL-1615RGBC-WS2812B, symbol PCM_JLCPCB-Extended:LED, WS2812B, 1615
- added D2: LED, PCM_JLCPCB:D_0603, symbol Device:LED
- added D3: Yellow, PCM_JLCPCB:D_0603, symbol PCM_JLCPCB-Diodes:LED,0603,Yellow
- added R23: 180Ω, PCM_JLCPCB:R_0603, symbol PCM_JLCPCB-Resistors:0603,180Ω
- added R24: 560Ω, PCM_JLCPCB:R_0603, symbol PCM_JLCPCB-Resistors:0603,560Ω
- TP8, TP9: footprint TestPoint:TestPoint_Pad_D1.5mm -> TestPoint:TestPoint_Pad_D1.0mm
Connections:
- net +3V3: now also R23.2, R24.2
- net GP10: now also D3.1
- net GP9: now also D2.1 (K)
- new net: D3.2, R24.1
- new net: D2.2 (A), R23.1
