File: pumper/pumper.kicad_pcb (KiCad board)
At the start: 4 copper layers, 33.8 x 93.1 mm, 90 parts, among them J1 Connector, USB-TYPE-C-16P, J2 Conn_01x03, J3 AudioJack4, SW1 1TS015A-1400-0600-CT, SW2 1TS015A-1400-0600-CT, U1 TLV76733DRVx, U2 TLV76733DRVx, U3 LM27762, U4 RP2354A-QFN60, U5 ABM8-272-T3_C20625731, U6 OPA1652AIDR, U7 PCM5102A, U8 OPA1622IDRCR

Commit message: feat: update kicad source files
Parts:
- C9: value 4.7uF -> 470nF
- moved C27 7.85 mm to (138.2, 118.3)
- moved C28 7.85 mm to (138.2, 117.4)
- moved C32 4.88 mm to (132.1, 112.0), turned to 0 degrees
- moved C31 4.62 mm to (132.1, 111.1), turned to 0 degrees
- moved C33 3.18 mm to (129.8, 123.8)
- moved C34 3.18 mm to (129.8, 124.7)
- moved C35 3.18 mm to (137.4, 123.8)
- moved C36 3.18 mm to (126.7, 120.6)
- moved R14 3.18 mm to (127.9, 120.6)
- moved R15 3.18 mm to (137.4, 121.8)
- moved U6 3.18 mm to (132.6, 120.4)
- moved D3 2.55 mm to (130.9, 140.8)
- moved C3 1.30 mm to (129.1, 62.5)
- moved R2 1.30 mm to (129.1, 61.6)
- renumbered C44 to C31, C31 to C32, C32 to C33, C33 to C34, C34 to C35, C35 to C36, C36 to C37, C37 to C38, C38 to C39, C39 to C40, C40 to C41, C41 to C42, C42 to C43, C43 to C44, D2 to D1, D4 to D2, D5 to D3
Routing:
- net Net-(U7-OUTR): track 15.9 -> 24.1 mm
- net /Audio processing/1652OUTR: track 70.0 -> 73.9 mm
- net Net-(U7-OUTL): track 10.3 -> 13.4 mm
- net /Audio processing/OUTR: track 25.7 -> 28.8 mm
- net /Audio processing/VOLOUTR: track 30.2 -> 27.2 mm
- net -4V5: track 56.7 -> 58.9 mm
- net VBUS: track 94.6 -> 92.4 mm
- net +4V5: track 59.8 -> 61.8 mm
- net +AUDIO_3V3: track 33.4 -> 35.1 mm
- net /Audio processing/5102AVDD: track 6.34 -> 4.75 mm
- net Net-(J1-CC2): track 4.94 -> 3.62 mm
- net /Audio processing/1652OUTL: track 71.3 -> 70.1 mm
- net GND: track 70.5 -> 70.3 mm, vias 144 -> 153

Commit message: feat: update design files
Parts:
- removed the J2 at (129.2, 93.8)
- added C11: 2.2uF, PCM_JLCPCB:C_0603, F.Cu at (146.0, 57.4)
- added C27: 100nF, PCM_JLCPCB:C_0402, F.Cu at (147.7, 144.1)
- added C28: 100nF, PCM_JLCPCB:C_0402, F.Cu at (144.1, 144.1)
- added D2: WS2812B, PCM_JLCPCB:LED-SMD_4P-L1.6-W1.5_XL-1615RGBC-WS2812B, F.Cu at (144.4, 142.7)
- added D3: WS2812B, PCM_JLCPCB:LED-SMD_4P-L1.6-W1.5_XL-1615RGBC-WS2812B, F.Cu at (148.0, 142.7)
- added R14: 2kΩ, PCM_JLCPCB:R_0402, F.Cu at (139.0, 122.3)
- added R15: 2kΩ, PCM_JLCPCB:R_0402, F.Cu at (126.2, 122.2)
- added TP1: TestPoint, TestPoint:TestPoint_Pad_D1.5mm, B.Cu at (133.6, 63.0)
- added TP2: TestPoint, TestPoint:TestPoint_Pad_D1.5mm, B.Cu at (135.9, 69.6)
- added TP3: TestPoint, TestPoint:TestPoint_Pad_D1.5mm, B.Cu at (131.9, 69.6)
- added TP4: TestPoint, TestPoint:TestPoint_Pad_D1.5mm, B.Cu at (140.9, 95.3)
- added TP5: TestPoint, TestPoint:TestPoint_Pad_D1.5mm, B.Cu at (127.2, 103.4)
- added TP6: TestPoint, TestPoint:TestPoint_Pad_D1.5mm, B.Cu at (140.9, 104.4)
- added TP7: TestPoint, TestPoint:TestPoint_Pad_D1.5mm, B.Cu at (140.9, 101.4)
- added TP8: TestPoint, TestPoint:TestPoint_Pad_D1.5mm, B.Cu at (131.4, 89.0)
- added TP9: TestPoint, TestPoint:TestPoint_Pad_D1.5mm, B.Cu at (134.3, 89.0)
- C6: value 10uF -> 2.2uF; footprint PCM_JLCPCB:C_0402 -> PCM_JLCPCB:C_0603
- C7: value 1uF -> 4.7uF
- C9: value 470nF -> 1uF
- moved C10 52.5 mm to (149.1, 58.5), turned to 0 degrees
- moved C7 50.6 mm to (150.0, 60.4)
- moved R4 50.3 mm to (149.1, 61.3), turned to 0 degrees
- moved R3 49.7 mm to (149.1, 62.2), turned to 180 degrees
- moved C6 47.8 mm to (141.6, 62.9), turned to -90 degrees
- moved U3 47.2 mm to (145.7, 60.3), turned to 180 degrees
- moved R6 46.6 mm to (143.1, 57.6), turned to 0 degrees
- moved R7 45.8 mm to (143.1, 58.5), turned to 180 degrees
- moved C9 44.0 mm to (142.9, 60.3), turned to 90 degrees
- moved R5 42.6 mm to (141.7, 60.3), turned to -90 degrees
- moved C8 41.7 mm to (140.8, 60.3), turned to 90 degrees
- moved C5 5.21 mm to (126.0, 102.8), turned to 180 degrees
- moved C4 4.97 mm to (124.8, 97.7), turned to -90 degrees
- moved C33 4.23 mm to (128.4, 103.2)
- moved C32 4.23 mm to (129.5, 110.4)
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- renumbered C11 to C12, C12 to C13, C13 to C14, C14 to C15, C15 to C16, C16 to C17, C17 to C18, C18 to C19, C19 to C20, C20 to C21, C21 to C22, C22 to C23, C23 to C24, C24 to C25, C25 to C26, C26 to C29, C27 to C30, C28 to C31, C29 to C32, C30 to C33, C31 to C34, C32 to C35, C33 to C36, C34 to C37, C35 to C38, C36 to C39, C37 to C40, C38 to C41, C39 to C42, C40 to C43, C41 to C44, C42 to C45, C43 to C46, C44 to C47, D2 to D4, D3 to D5, J3 to J2, R14 to R16, R15 to R17, R16 to R18, R17 to R19, R18 to R20, R19 to R21, R20 to R22
Connections:
- C6 pad 1: VBUS -> +4V5
Routing:
- net /MCU/GP12: track 0.00 -> 78.4 mm, vias 0 -> 2
- net VBUS: track 92.4 -> 156.8 mm, vias 6 -> 10
- net +4V5: track 61.8 -> 124.9 mm, vias 5 -> 7
- net -4V5: track 58.9 -> 118.5 mm, vias 4 -> 5
- net GND: track 70.3 -> 97.9 mm, vias 153 -> 146
- net /MCU/RUN: track 53.8 -> 45.5 mm
- net /MCU/SWCLK: track 14.3 -> 8.15 mm, vias 0 -> 1
- net +3V3: track 35.1 -> 40.7 mm
- net Net-(U7-OUTR): track 24.1 -> 18.6 mm
- net /Audio processing/1652OUTR: track 73.9 -> 68.5 mm
- net Net-(U7-LDOO): track 7.76 -> 3.00 mm
- net GP21: track 31.8 -> 28.1 mm
- net /MCU/SWDIO: track 10.4 -> 6.75 mm, vias 0 -> 1
- net GP20: track 31.3 -> 27.7 mm
- net GP19: track 32.5 -> 29.2 mm
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Other:
- outline, holes or cut-outs redrawn
- board text added: "3.5mm Headphone"
- board text added: "RP2350 PCM5120A OPA1652 OPA1622"
- board text added: "USB C"
- board text added: "wolf-yuan.dev"

Commit message: feat: update kicad files
Parts:
- removed C27, C28: 100nF, PCM_JLCPCB:C_0402
- added R23: 180Ω, PCM_JLCPCB:R_0603, F.Cu at (147.0, 142.8)
- added R24: 560Ω, PCM_JLCPCB:R_0603, F.Cu at (143.5, 142.8)
- D2: value WS2812B -> LED; footprint PCM_JLCPCB:LED-SMD_4P-L1.6-W1.5_XL-1615RGBC-WS2812B -> PCM_JLCPCB:D_0603
- D3: value WS2812B -> Yellow; footprint PCM_JLCPCB:LED-SMD_4P-L1.6-W1.5_XL-1615RGBC-WS2812B -> PCM_JLCPCB:D_0603
- TP1, TP2, TP3, TP4, TP5, TP6, TP7, TP8, TP9: footprint TestPoint:TestPoint_Pad_D1.5mm -> TestPoint:TestPoint_Pad_D1.0mm
- moved D2 4.20 mm to (148.6, 142.6), turned to -90 degrees
- moved D3 2.90 mm to (145.1, 142.6), turned to -90 degrees
- moved C18 2.35 mm to (128.2, 86.2), turned to 180 degrees
Connections:
- D2 pad 1: Net-(D2-DOUT) -> /MCU/GP9
- D2 pad 2: VBUS -> Net-(D2-A)
- D3 pad 1: unconnected-(D3-DOUT-Pad1) -> /MCU/GP10
- D3 pad 2: VBUS -> Net-(D3-Pad2)
Routing:
- net /MCU/GP9: track 0.00 -> 87.6 mm, vias 0 -> 2
- net +3V3: track 40.7 -> 125.1 mm, vias 10 -> 12
- net /MCU/GP10: track 0.00 -> 83.9 mm, vias 0 -> 2
- net /MCU/GP12: track 78.4 -> 0.00 mm, vias 2 -> 0
- net VBUS: track 156.8 -> 87.2 mm, vias 10 -> 7
- net GND: track 97.9 -> 94.5 mm, vias 146 -> 153
- net Net-(D2-DOUT): track 2.78 -> 0.00 mm
- net Net-(D3-Pad2): track 0.00 -> 1.70 mm
- net Net-(D2-A): track 0.00 -> 1.70 mm
Other:
- board text added: "LM27761"
- board text added: "PCM5102A"
- board text added: "RP2354A"
