File: pumper/pumper.kicad_sch (KiCad schematic)
At the start: 29 parts, among them J1 Connector, USB-TYPE-C-16P, U1 TLV76733DRVx, U2 TLV76733DRVx, U3 LM27762

Commit message: feat: update kicad source files
Parts:
- C9: value 4.7uF -> 470nF; symbol PCM_JLCPCB-Capacitors:0402,4.7uF -> PCM_JLCPCB-Capacitors:0402,470nF; Attrition Qty 10 -> 12; Capacitance 4.7uF -> 470nF; Class Basic Component -> Preferred Component; LCSC C23733 -> C47339; Part CL05A475MP5NRNC -> CL05A474KP5NNNC; Price 0.008USD -> 0.007USD; Stock 4366811 -> 84633; Tolerance ±20% -> ±10%
- renumbered D2 to D1
Changed lines of the file:
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@@
 	)
 	(symbol
-		(lib_id "PCM_JLCPCB-Capacitors:0402,4.7uF")
+		(lib_id "PCM_JLCPCB-Capacitors:0402,470nF")
 		(at 180.34 125.73 0)
 		(unit 1)
@@
 			)
 		)
-		(property "Value" "4.7uF"
+		(property "Value" "470nF"
 			(at 182.88 125.73 0)
 			(effects
@@
 			)
 		)
-		(property "Datasheet" "https://www.lcsc.com/datasheet/lcsc_datasheet_2304140030_Samsung-Electro-Mechanics-CL05A475MP5NRNC_C23733.pdf"
+		(property "Datasheet" "https://www.lcsc.com/datasheet/lcsc_datasheet_2304140030_Samsung-Electro-Mechanics-CL05A474KP5NNNC_C47339.pdf"
 			(at 180.34 125.73 0)
 			(effects
@@
 			)
 		)
-		(property "Description" "10V 4.7uF X5R ±20% 0402 Multilayer Ceramic Capacitors MLCC - SMD/SMT ROHS"
+		(property "Description" "10V 470nF X5R ±10% 0402 Multilayer Ceramic Capacitors MLCC - SMD/SMT ROHS"
 			(at 180.34 125.73 0)
 			(effects
@@
 			)
 		)
-		(property "LCSC" "C23733"
+		(property "LCSC" "C47339"
 			(at 180.34 125.73 0)
 			(effects
@@
 			)
 		)
-		(property "Stock" "4366811"
+		(property "Stock" "84633"
 			(at 180.34 125.73 0)
 			(effects
@@
 			)
 		)
-		(property "Price" "0.008USD"
+		(property "Price" "0.007USD"
 			(at 180.34 125.73 0)
 			(effects
@@
 			)
 		)
-		(property "Attrition Qty" "10"
+		(property "Attrition Qty" "12"
 			(at 180.34 125.73 0)
 			(effects
@@
 			)
 		)
-		(property "Class" "Basic Component"
+		(property "Class" "Preferred Component"
 			(at 180.34 125.73 0)
 			(effects
@@
 			)
 		)
-		(property "Part" "CL05A475MP5NRNC"
+		(property "Part" "CL05A474KP5NNNC"
 			(at 180.34 125.73 0)
 			(effects
@@
 			)
 		)
-		(property "Tolerance" "±20%"
+		(property "Tolerance" "±10%"
 			(at 180.34 125.73 0)
 			(effects
@@
 			)
 		)
-		(property "Capacitance" "4.7uF"
+		(property "Capacitance" "470nF"
 			(at 180.34 125.73 0)
 			(effects
@@
 		(dnp no)
 		(fields_autoplaced yes)
-		(property "Reference" "D2"
+		(property "Reference" "D1"
 			(at 120.65 25.4 0)
 			(effects
@@
 			(project ""
 				(path "/ff072219-444d-4fc6-9bb4-21a48733c6c1"
-					(reference "D2")
+					(reference "D1")
 					(unit 1)
 				)

Commit message: feat: update design files
Parts:
- removed C6: 10uF, PCM_JLCPCB:C_0402, symbol PCM_JLCPCB-Capacitors:0402,10uF
- removed C7: 1uF, PCM_JLCPCB:C_0402, symbol PCM_JLCPCB-Capacitors:0402,1uF
- added C11, C6: 2.2uF, PCM_JLCPCB:C_0603, symbol PCM_JLCPCB-Capacitors:0603,2.2uF
- added C7: 4.7uF, PCM_JLCPCB:C_0402, symbol PCM_JLCPCB-Capacitors:0402,4.7uF
- added TP1, TP2, TP3, TP4, TP5, TP6, TP7: TestPoint, TestPoint:TestPoint_Pad_D1.5mm, symbol Connector:TestPoint
- C9: value 470nF -> 1uF; symbol PCM_JLCPCB-Capacitors:0402,470nF -> PCM_JLCPCB-Capacitors:0402,1uF; Attrition Qty 12 -> 10; Capacitance 470nF -> 1uF; Class Preferred Component -> Basic Component; LCSC C47339 -> C52923; Part CL05A474KP5NNNC -> CL05A105KA5NQNC; Price 0.007USD -> 0.006USD; Stock 84633 -> 7021828; Voltage Rated 10V -> 25V
Connections:
- net +3V3: now also TP2.1
- net +4V5: now also C6.1, TP6.1
- net +AUDIO_3V3: now also TP5.1
- net -4V5: now also C11.1, TP7.1
- net GND: now also C11.2, C6.2, C7.2, TP4.1
- net VBUS: now also C7.1, TP3.1
- net at F1.1, J1.A9B4 (VBUS), J1.B9A4 (VBUS): now also TP1.1
Other:
- moved on the sheet: F1

Commit message: feat: update kicad files
Parts:
- TP1, TP2, TP3, TP4, TP5, TP6, TP7: footprint TestPoint:TestPoint_Pad_D1.5mm -> TestPoint:TestPoint_Pad_D1.0mm
Changed lines of the file:
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@@
 			)
 		)
-		(property "Footprint" "TestPoint:TestPoint_Pad_D1.5mm"
+		(property "Footprint" "TestPoint:TestPoint_Pad_D1.0mm"
 			(at 264.16 127 0)
 			(effects
@@
 			)
 		)
-		(property "Footprint" "TestPoint:TestPoint_Pad_D1.5mm"
+		(property "Footprint" "TestPoint:TestPoint_Pad_D1.0mm"
 			(at 264.16 97.79 0)
 			(effects
@@
 			)
 		)
-		(property "Footprint" "TestPoint:TestPoint_Pad_D1.5mm"
+		(property "Footprint" "TestPoint:TestPoint_Pad_D1.0mm"
 			(at 55.88 21.59 0)
 			(effects
@@
 			)
 		)
-		(property "Footprint" "TestPoint:TestPoint_Pad_D1.5mm"
+		(property "Footprint" "TestPoint:TestPoint_Pad_D1.0mm"
 			(at 260.35 25.4 0)
 			(effects
@@
 			)
 		)
-		(property "Footprint" "TestPoint:TestPoint_Pad_D1.5mm"
+		(property "Footprint" "TestPoint:TestPoint_Pad_D1.0mm"
 			(at 74.93 53.34 0)
 			(effects
@@
 			)
 		)
-		(property "Footprint" "TestPoint:TestPoint_Pad_D1.5mm"
+		(property "Footprint" "TestPoint:TestPoint_Pad_D1.0mm"
 			(at 260.35 60.96 0)
 			(effects
@@
 			)
 		)
-		(property "Footprint" "TestPoint:TestPoint_Pad_D1.5mm"
+		(property "Footprint" "TestPoint:TestPoint_Pad_D1.0mm"
 			(at 60.96 53.34 0)
 			(effects
