File: feather/feather.kicad_pcb (KiCad board)
At the start: 4 copper layers, 61.4 x 38.8 mm, 146 parts, among them CN1 ST-0337D00-071-1A2H, CN2 GT-3321667P-01, J1 Connector, USB-TYPE-C-16P, SW1 1TS015A-1400-0600-CT, SW2 1TS015A-1400-0600-CT, U1 TLV76733DRVx, U10 OPA1622, U11 OPA1622, U2 LM27762, U3 TAD5242IRGER, U4 TLV76733DRVx, U5 OPA1612AxD, U6 RP2350A-QFN60, U7 OPA1612AxD, U8 OPA1612AxD, U9 OPA1622, X1 12MHz

Commit message: feat: update feather design files
Routing:
- net +3V3: track 146.7 -> 143.8 mm, vias 11 -> 13
- net /GP10: track 59.1 -> 61.5 mm
- net /BAL-1622-EN: track 71.1 -> 72.7 mm
- net +AUDIO3V3: track 23.8 -> 25.0 mm
- net /OUT-BAL-1N: track 20.3 -> 21.4 mm
- net /1612-UNBAL-1: track 26.0 -> 24.9 mm
- net +1V1: track 59.9 -> 61.0 mm
- net Net-(U5A--): track 7.82 -> 6.98 mm
- net GND: track 49.0 -> 49.2 mm, vias 309 -> 288
Other:
- outline, holes or cut-outs redrawn
- board text added: "Balanced"
- board text added: "Portable USB DAC Card"
- board text added: "Unbalanced"
- board text removed: "USB-C"
